File: nuc64-debug.kicad_pcb (KiCad board)
At the start: 2 copper layers, 17.1 x 30.5 mm, 24 parts, among them J1 SWD, J2 POW, SW1 BOOT, SW2 RST

Commit message: Updated BOM
Routing:
- net GND: track 101.1 -> 116.0 mm, vias 7 -> 9
Changed lines of the file:
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@@
+	)
+	(segment
+		(start 123.5 87.4)
+		(end 123.5 86.9)
+		(width 0.3)
+		(layer "F.Cu")
+		(net 5)
 	)
 	(segment
@@
 	(segment
 		(start 122.265 87.44)
+		(end 123.46 87.44)
+		(width 0.3)
+		(layer "F.Cu")
+		(net 5)
+	)
+	(segment
+		(start 122.265 87.44)
 		(end 119.825 87.44)
 		(width 0.25)
@@
 	)
 	(segment
+		(start 123.5 86.9)
+		(end 123.9 86.5)
+		(width 0.3)
+		(layer "F.Cu")
+		(net 5)
+	)
+	(segment
+		(start 123.9 86.5)
+		(end 124.4 86.5)
+		(width 0.3)
+		(layer "F.Cu")
+		(net 5)
+	)
+	(segment
 		(start 122.265 90.565)
 		(end 122.1 90.4)
@@
 	)
 	(segment
+		(start 125.1 86.2)
+		(end 124.7 86.2)
+		(width 0.3)
+		(layer "F.Cu")
+		(net 5)
+	)
+	(segment
+		(start 124.4 86.5)
+		(end 124.7 86.2)
+		(width 0.3)
+		(layer "F.Cu")
+		(net 5)
+	)
+	(segment
+		(start 123.46 87.44)
+		(end 123.5 87.4)
+		(width 0.3)
+		(layer "F.Cu")
+		(net 5)
+	)
+	(segment
 		(start 110 76.734884)
 		(end 109.982558 76.717442)
@@
 	)
 	(via
+		(at 124.9 74.5)
+		(size 0.45)
+		(drill 0.3)
+		(layers "F.Cu" "B.Cu")
+		(net 5)
+	)
+	(via
+		(at 125.1 86.2)
+		(size 0.45)
+		(drill 0.3)
+		(layers "F.Cu" "B.Cu")
+		(net 5)
+	)
+	(via
 		(at 122.1 90.4)
 		(size 0.45)
@@
 	)
 	(segment
+		(start 118.7 69.5)
+		(end 118.4025 69.2025)
+		(width 0.3)
+		(layer "B.Cu")
+		(net 5)
+	)
+	(segment
 		(start 120.7 94.826)
 		(end 120.7 96.1)
@@
 	)
 	(segment
+		(start 119.8 69.5)
+		(end 118.7 69.5)
+		(width 0.3)
+		(layer "B.Cu")
+		(net 5)
+	)
+	(segment
+		(start 120.8 70.1)
+		(end 120.5 69.8)
+		(width 0.3)
+		(layer "B.Cu")
+		(net 5)
+	)
+	(segment
+		(start 124.9 74.5)
+		(end 122.9 74.5)
+		(width 0.3)
+		(layer "B.Cu")
+		(net 5)
+	)
+	(segment
 		(start 110.49 76.11)
 		(end 109.882558 76.717442)
@@
 	)
 	(segment
+		(start 120.5 69.8)
+		(end 120.1 69.8)
+		(width 0.3)
+		(layer "B.Cu")
+		(net 5)
+	)
+	(segment
+		(start 120.1 69.8)
+		(end 119.8 69.5)
+		(width 0.3)
+		(layer "B.Cu")
+		(net 5)
+	)
+	(segment
 		(start 110.49 68.58)
 		(end 118.11 76.2)
@@
 	)
 	(segment
+		(start 120.8 72.4)
+		(end 120.8 70.1)
+		(width 0.3)
+		(layer "B.Cu")
+		(net 5)
+	)
+	(segment
 		(start 114.825 96.4)
 		(end 116.5125 94.7125)
@@
 	)
 	(segment
+		(start 118.4025 69.2025)
+		(end 118.4025 67.945)
+		(width 0.3)
+		(layer "B.Cu")
+		(net 5)
+	)
+	(segment
 		(start 110.49 68.58)
 		(end 110.49 76.11)
 		(width 0.3)
 		(layer "B.Cu")
+		(net 5)
+	)
+	(segment
+		(start 122.9 74.5)
+		(end 120.8 72.4)
+		(width 0.3)
+		(layer "B.Cu")
